File: main.brd (EAGLE design)
At the start: 35.6 x 50.8 mm, 12 parts

Commit message: Replaced incorrect component and converted README to Markdown
Replaced NOR gates with NAND gates to match AMIS schematic and updated parts list to reflect the change.
Parts:
- NAND: value 4001N -> 4011N
- renumbered NOR to NAND
Changed lines of the file:
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@@
 </autorouter>
 <elements>
-<element name="NOR" library="40xx" package="DIL14" value="4001N" x="17.78" y="29.845" smashed="yes" rot="R270">
+<element name="NAND" library="40xx" package="DIL14" value="4011N" x="17.78" y="29.845" smashed="yes" rot="R270">
 <attribute name="VALUE" x="17.145" y="29.845" size="1.27" layer="27" font="vector" rot="R90" align="top-center"/>
 </element>
@@
 <signal name="VCC">
 <contactref element="LD117AV33" pad="2"/>
-<contactref element="NOR" pad="14"/>
+<contactref element="NAND" pad="14"/>
 <contactref element="INV" pad="14"/>
 <contactref element="ICSP" pad="1"/>
@@
 <contactref element="ICSP" pad="2"/>
 <contactref element="ISO1" pad="4"/>
-<contactref element="NOR" pad="7"/>
+<contactref element="NAND" pad="7"/>
 <contactref element="INV" pad="7"/>
 <contactref element="C1" pad="2"/>
@@
 </signal>
 <signal name="N$3">
-<contactref element="NOR" pad="6"/>
+<contactref element="NAND" pad="6"/>
 <contactref element="INV" pad="8"/>
 <wire x1="13.97" y1="24.765" x2="17.78" y2="20.955" width="0.254" layer="16"/>
@@
 </signal>
 <signal name="N$4">
-<contactref element="NOR" pad="2"/>
+<contactref element="NAND" pad="2"/>
 <contactref element="INV" pad="2"/>
 <wire x1="13.97" y1="34.925" x2="15.24" y2="34.925" width="0.254" layer="16"/>
@@
 </signal>
 <signal name="N$5">
-<contactref element="NOR" pad="8"/>
+<contactref element="NAND" pad="8"/>
 <contactref element="INV" pad="4"/>
 <wire x1="21.59" y1="22.225" x2="23.495" y2="24.13" width="0.254" layer="16"/>
@@
 </signal>
 <signal name="N$6">
-<contactref element="NOR" pad="12"/>
+<contactref element="NAND" pad="12"/>
 <contactref element="INV" pad="6"/>
 <wire x1="22.86" y1="31.115" x2="21.59" y2="32.385" width="0.254" layer="16"/>
@@
 </signal>
 <signal name="N$7">
-<contactref element="NOR" pad="11"/>
-<contactref element="NOR" pad="9"/>
+<contactref element="NAND" pad="11"/>
+<contactref element="NAND" pad="9"/>
 <contactref element="INV" pad="1"/>
 <wire x1="25.4" y1="37.465" x2="23.495" y2="35.56" width="0.254" layer="1"/>
@@
 </signal>
 <signal name="N$8">
-<contactref element="NOR" pad="4"/>
+<contactref element="NAND" pad="4"/>
 <contactref element="INV" pad="3"/>
-<contactref element="NOR" pad="1"/>
+<contactref element="NAND" pad="1"/>
 <wire x1="15.24" y1="36.195" x2="26.67" y2="36.195" width="0.254" layer="16"/>
 <wire x1="27.305" y1="34.29" x2="25.4" y2="32.385" width="0.254" layer="16"/>
@@
 </signal>
 <signal name="N$22">
-<contactref element="NOR" pad="13"/>
+<contactref element="NAND" pad="13"/>
 <wire x1="19.05" y1="24.765" x2="19.05" y2="32.385" width="0.254" layer="1"/>
 <wire x1="21.59" y1="34.925" x2="19.05" y2="32.385" width="0.254" layer="1"/>
@@
 </signal>
 <signal name="N$21">
-<contactref element="NOR" pad="5"/>
+<contactref element="NAND" pad="5"/>
 <contactref element="MSP430G2553" pad="8"/>
 <wire x1="13.97" y1="27.305" x2="12.065" y2="25.4" width="0.254" layer="1"/>
@@
 </signal>
 <signal name="N$24">
-<contactref element="NOR" pad="3"/>
+<contactref element="NAND" pad="3"/>
 <contactref element="ISO2" pad="3"/>
 <contactref element="MSP430G2553" pad="9"/>
@@
 </signal>
 <signal name="N$25">
-<contactref element="NOR" pad="10"/>
+<contactref element="NAND" pad="10"/>
 <contactref element="ISO1" pad="3"/>
 <contactref element="MSP430G2553" pad="12"/>
