File: main.sch (EAGLE design)
At the start: 12 parts

Commit message: Replaced incorrect component and converted README to Markdown
Replaced NOR gates with NAND gates to match AMIS schematic and updated parts list to reflect the change.
Parts:
- removed NOR: 4001N, 40xx:4001N
- added NAND: 4011N, 40xx:4011N
Connections:
- net GND: now also NANDP.VSS; no longer NORP.VSS
- net N$21: now also NANDB.I0; no longer NORB.I0
- net N$22: now also NANDD.I1; no longer NORD.I1
- net N$24: now also NANDA.O; no longer NORA.O
- net N$25: now also NANDC.O; no longer NORC.O
- net N$3: now also NANDB.I1; no longer NORB.I1
- net N$4: now also NANDA.I1; no longer NORA.I1
- net N$5: now also NANDC.I0; no longer NORC.I0
- net N$6: now also NANDD.I0; no longer NORD.I0
- net N$7: now also NANDC.I1, NANDD.O; no longer NORC.I1, NORD.O
- net N$8: now also NANDA.I0, NANDB.O; no longer NORA.I0, NORB.O
- net VCC: now also NANDP.VDD; no longer NORP.VDD
Changed lines of the file:
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@@
 </classes>
 <parts>
-<part name="NOR" library="40xx" deviceset="4001" device="N"/>
+<part name="NAND" library="40xx" deviceset="4011" device="N"/>
 <part name="INV" library="40xx" deviceset="4069" device="N"/>
 <part name="ISO1" library="texas" deviceset="ISO1050" device="DUB" value=""/>
@@
 </plain>
 <instances>
-<instance part="NOR" gate="A" x="86.36" y="86.36" rot="R180"/>
-<instance part="NOR" gate="B" x="86.36" y="55.88"/>
-<instance part="NOR" gate="C" x="160.02" y="86.36"/>
-<instance part="NOR" gate="D" x="160.02" y="55.88" rot="R180"/>
+<instance part="NAND" gate="A" x="86.36" y="86.36" rot="R180"/>
+<instance part="NAND" gate="B" x="86.36" y="55.88"/>
+<instance part="NAND" gate="C" x="160.02" y="86.36"/>
+<instance part="NAND" gate="D" x="160.02" y="55.88" rot="R180"/>
 <instance part="INV" gate="A" x="106.68" y="88.9" rot="R180"/>
 <instance part="INV" gate="B" x="139.7" y="88.9"/>
@@
 <instance part="P+1" gate="VCC" x="43.18" y="55.88"/>
 <instance part="GND1" gate="1" x="25.4" y="35.56"/>
-<instance part="NOR" gate="P" x="17.78" y="17.78"/>
+<instance part="NAND" gate="P" x="17.78" y="17.78"/>
 <instance part="INV" gate="P" x="33.02" y="17.78"/>
 <instance part="P+2" gate="VCC" x="17.78" y="27.94"/>
@@
 </segment>
 <segment>
-<pinref part="NOR" gate="P" pin="VDD"/>
+<pinref part="NAND" gate="P" pin="VDD"/>
 <pinref part="P+2" gate="VCC" pin="VCC"/>
 </segment>
@@
 </segment>
 <segment>
-<pinref part="NOR" gate="P" pin="VSS"/>
+<pinref part="NAND" gate="P" pin="VSS"/>
 <pinref part="GND6" gate="1" pin="GND"/>
 </segment>
@@
 <net name="N$3" class="0">
 <segment>
-<pinref part="NOR" gate="B" pin="I1"/>
+<pinref part="NAND" gate="B" pin="I1"/>
 <pinref part="INV" gate="D" pin="O"/>
 <wire x1="73.66" y1="53.34" x2="78.74" y2="53.34" width="0.1524" layer="91"/>
@@
 <net name="N$4" class="0">
 <segment>
-<pinref part="NOR" gate="A" pin="I1"/>
+<pinref part="NAND" gate="A" pin="I1"/>
 <pinref part="INV" gate="A" pin="O"/>
 <wire x1="96.52" y1="88.9" x2="93.98" y2="88.9" width="0.1524" layer="91"/>
@@
 <net name="N$5" class="0">
 <segment>
-<pinref part="NOR" gate="C" pin="I0"/>
+<pinref part="NAND" gate="C" pin="I0"/>
 <pinref part="INV" gate="B" pin="O"/>
 <wire x1="149.86" y1="88.9" x2="152.4" y2="88.9" width="0.1524" layer="91"/>
@@
 <net name="N$6" class="0">
 <segment>
-<pinref part="NOR" gate="D" pin="I0"/>
+<pinref part="NAND" gate="D" pin="I0"/>
 <pinref part="INV" gate="C" pin="O"/>
 <wire x1="172.72" y1="53.34" x2="167.64" y2="53.34" width="0.1524" layer="91"/>
@@
 <net name="N$7" class="0">
 <segment>
-<pinref part="NOR" gate="D" pin="O"/>
-<pinref part="NOR" gate="C" pin="I1"/>
+<pinref part="NAND" gate="D" pin="O"/>
+<pinref part="NAND" gate="C" pin="I1"/>
 <wire x1="152.4" y1="55.88" x2="152.4" y2="83.82" width="0.1524" layer="91"/>
 <pinref part="INV" gate="A" pin="I"/>
@@
 <net name="N$8" class="0">
 <segment>
-<pinref part="NOR" gate="B" pin="O"/>
+<pinref part="NAND" gate="B" pin="O"/>
 <pinref part="INV" gate="B" pin="I"/>
 <wire x1="93.98" y1="55.88" x2="114.3" y2="55.88" width="0.1524" layer="91"/>
 <wire x1="114.3" y1="55.88" x2="129.54" y2="88.9" width="0.1524" layer="91"/>
-<pinref part="NOR" gate="A" pin="I0"/>
+<pinref part="NAND" gate="A" pin="I0"/>
 <wire x1="93.98" y1="55.88" x2="93.98" y2="83.82" width="0.1524" layer="91"/>
 <junction x="93.98" y="55.88"/>
@@
 <net name="N$25" class="0">
 <segment>
-<pinref part="NOR" gate="C" pin="O"/>
+<pinref part="NAND" gate="C" pin="O"/>
 <pinref part="ISO1" gate="G$1" pin="TXD"/>
 <wire x1="167.64" y1="86.36" x2="172.72" y2="81.28" width="0.1524" layer="91"/>
@@
 <net name="N$24" class="0">
 <segment>
-<pinref part="NOR" gate="A" pin="O"/>
+<pinref part="NAND" gate="A" pin="O"/>
 <pinref part="ISO2" gate="G$1" pin="TXD"/>
 <wire x1="78.74" y1="86.36" x2="66.04" y2="86.36" width="0.1524" layer="91"/>
@@
 <net name="N$21" class="0">
 <segment>
-<pinref part="NOR" gate="B" pin="I0"/>
+<pinref part="NAND" gate="B" pin="I0"/>
 <wire x1="99.06" y1="20.32" x2="76.2" y2="20.32" width="0.1524" layer="91"/>
 <wire x1="76.2" y1="20.32" x2="76.2" y2="58.42" width="0.1524" layer="91"/>
@@
 <net name="N$22" class="0">
 <segment>
-<pinref part="NOR" gate="D" pin="I1"/>
+<pinref part="NAND" gate="D" pin="I1"/>
 <wire x1="147.32" y1="20.32" x2="205.74" y2="20.32" width="0.1524" layer="91"/>
 <wire x1="167.64" y1="58.42" x2="205.74" y2="58.42" width="0.1524" layer="91"/>
